File: selftest_bd/relay_driver.kicad_sch (KiCad schematic)
At the start: 63 parts, among them K1 TQ2-5_Split, K10 TQ2-5_Split, K11 TQ2-5_Split, K12 TQ2-5_Split, K13 TQ2-5_Split, K14 TQ2-5_Split, K15 TQ2-5_Split, K16 TQ2-5_Split, K17 TQ2-5_Split, K2 TQ2-5_Split, K3 TQ2-5_Split, K4 TQ2-5_Split, K5 TQ2-5_Split, K6 TQ2-5_Split, K7 TQ2-5_Split, K8 TQ2-5_Split, K9 TQ2-5_Split, U2 ULN2003A, U3 ULN2003A

Commit message: Commit V2.0
Redo PCB due to incorrect position of J1 and J2
Parts:
- renumbered K14 to K10, K15 to K11, K16 to K12, K10 to K13, K5 to K14, K4 to K15, K8 to K16, K7 to K2, K2 to K3, K12 to K4, K6 to K5, K11 to K6, K9 to K7, K13 to K8, K3 to K9
Other:
- title: FIRST TEST STATION SELFTEST BOARD 640-1010-010 -> FIRST TEST STATION SELFTEST BOARD 640-1010-020
Changed lines of the file:
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@@
   (paper "A")
   (title_block
-    (title "FIRST TEST STATION SELFTEST BOARD 640-1010-010")
-    (date "2023-05-16")
-    (rev "1.0")
+    (title "FIRST TEST STATION SELFTEST BOARD 640-1010-020")
+    (date "2023-10-01")
+    (rev "2.0")
   )
   (junction (at 110.49 147.32) (diameter 0) (color 0 0 0 0)
@@
   (symbol (lib_id "Library:TQ2-5_Split") (at 157.48 30.48 0) (unit 1)
     (in_bom yes) (on_board yes) (dnp no)
-    (property "Reference" "K2" (at 163.83 29.2099 0)
+    (property "Reference" "K3" (at 163.83 29.2099 0)
       (effects (font (size 1.27 1.27)) (justify left))
     )
@@
       (project "selftest_bd"
         (path "/e63e39d7-6ac0-4ffd-8aa3-1841a4541b55/3c0146c9-302b-4005-9f50-7766581fb71a"
-          (reference "K2") (unit 1)
+          (reference "K3") (unit 1)
         )
       )
@@
   (symbol (lib_id "Library:TQ2-5_Split") (at 176.53 30.48 0) (unit 1)
     (in_bom yes) (on_board yes) (dnp no)
-    (property "Reference" "K5" (at 182.88 29.2099 0)
+    (property "Reference" "K14" (at 182.88 29.2099 0)
       (effects (font (size 1.27 1.27)) (justify left))
     )
@@
       (project "selftest_bd"
         (path "/e63e39d7-6ac0-4ffd-8aa3-1841a4541b55/3c0146c9-302b-4005-9f50-7766581fb71a"
-          (reference "K5") (unit 1)
+          (reference "K14") (unit 1)
         )
       )
@@
   (symbol (lib_id "Library:TQ2-5_Split") (at 237.49 30.48 0) (unit 1)
     (in_bom yes) (on_board yes) (dnp no)
-    (property "Reference" "K7" (at 243.84 29.2099 0)
+    (property "Reference" "K2" (at 243.84 29.2099 0)
       (effects (font (size 1.27 1.27)) (justify left))
     )
@@
       (project "selftest_bd"
         (path "/e63e39d7-6ac0-4ffd-8aa3-1841a4541b55/3c0146c9-302b-4005-9f50-7766581fb71a"
-          (reference "K7") (unit 1)
+          (reference "K2") (unit 1)
         )
       )
@@
   (symbol (lib_id "Library:TQ2-5_Split") (at 215.9 83.82 0) (unit 1)
     (in_bom yes) (on_board yes) (dnp no)
-    (property "Reference" "K12" (at 222.25 82.5499 0)
+    (property "Reference" "K4" (at 222.25 82.5499 0)
       (effects (font (size 1.27 1.27)) (justify left))
     )
@@
       (project "selftest_bd"
         (path "/e63e39d7-6ac0-4ffd-8aa3-1841a4541b55/3c0146c9-302b-4005-9f50-7766581fb71a"
-          (reference "K12") (unit 1)
+          (reference "K4") (unit 1)
         )
       )
@@
   (symbol (lib_id "Library:TQ2-5_Split") (at 137.16 30.48 0) (unit 1)
     (in_bom yes) (on_board yes) (dnp no)
-    (property "Reference" "K9" (at 143.51 29.2099 0)
+    (property "Reference" "K7" (at 143.51 29.2099 0)
       (effects (font (size 1.27 1.27)) (justify left))
     )
@@
       (project "selftest_bd"
         (path "/e63e39d7-6ac0-4ffd-8aa3-1841a4541b55/3c0146c9-302b-4005-9f50-7766581fb71a"
-          (reference "K9") (unit 1)
+          (reference "K7") (unit 1)
         )
       )
@@
   (symbol (lib_id "Library:TQ2-5_Split") (at 195.58 83.82 0) (unit 1)
     (in_bom yes) (on_board yes) (dnp no)
-    (property "Reference" "K6" (at 201.93 82.5499 0)
+    (property "Reference" "K5" (at 201.93 82.5499 0)
       (effects (font (size 1.27 1.27)) (justify left))
     )
@@
       (project "selftest_bd"
         (path "/e63e39d7-6ac0-4ffd-8aa3-1841a4541b55/3c0146c9-302b-4005-9f50-7766581fb71a"
-          (reference "K6") (unit 1)
+          (reference "K5") (unit 1)
         )
       )
@@
   (symbol (lib_id "Library:TQ2-5_Split") (at 119.38 139.7 0) (unit 1)
     (in_bom yes) (on_board yes) (dnp no)
-    (property "Reference" "K15" (at 125.73 138.4299 0)
+    (property "Reference" "K11" (at 125.73 138.4299 0)
       (effects (font (size 1.27 1.27)) (justify left))
     )
@@
       (project "selftest_bd"
         (path "/e63e39d7-6ac0-4ffd-8aa3-1841a4541b55/3c0146c9-302b-4005-9f50-7766581fb71a"
-          (reference "K15") (unit 1)
+          (reference "K11") (unit 1)
         )
       )
@@
   (symbol (lib_id "Library:TQ2-5_Split") (at 116.84 30.48 0) (unit 1)
     (in_bom yes) (on_board yes) (dnp no)
-    (property "Reference" "K13" (at 123.19 29.2099 0)
+    (property "Reference" "K8" (at 123.19 29.2099 0)
       (effects (font (size 1.27 1.27)) (justify left))
     )
@@
       (project "selftest_bd"
         (path "/e63e39d7-6ac0-4ffd-8aa3-1841a4541b55/3c0146c9-302b-4005-9f50-7766581fb71a"
-          (reference "K13") (unit 1)
+          (reference "K8") (unit 1)
         )
       )
@@
   (symbol (lib_id "Library:TQ2-5_Split") (at 152.4 139.7 0) (unit 1)
     (in_bom yes) (on_board yes) (dnp no)
-    (property "Reference" "K16" (at 158.75 138.4299 0)
+    (property "Reference" "K12" (at 158.75 138.4299 0)
       (effects (font (size 1.27 1.27)) (justify left))
     )
@@
       (project "selftest_bd"
         (path "/e63e39d7-6ac0-4ffd-8aa3-1841a4541b55/3c0146c9-302b-4005-9f50-7766581fb71a"
-          (reference "K16") (unit 1)
+          (reference "K12") (unit 1)
         )
       )
@@
   (symbol (lib_id "Library:TQ2-5_Split") (at 215.9 30.48 0) (unit 1)
     (in_bom yes) (on_board yes) (dnp no)
-    (property "Reference" "K8" (at 222.25 29.2099 0)
+    (property "Reference" "K16" (at 222.25 29.2099 0)
       (effects (font (size 1.27 1.27)) (justify left))
     )
@@
       (project "selftest_bd"
         (path "/e63e39d7-6ac0-4ffd-8aa3-1841a4541b55/3c0146c9-302b-4005-9f50-7766581fb71a"
-          (reference "K8") (unit 1)
+          (reference "K16") (unit 1)
         )
       )
@@
   (symbol (lib_id "Library:TQ2-5_Split") (at 195.58 30.48 0) (unit 1)
     (in_bom yes) (on_board yes) (dnp no)
-    (property "Reference" "K4" (at 201.93 29.2099 0)
+    (property "Reference" "K15" (at 201.93 29.2099 0)
       (effects (font (size 1.27 1.27)) (justify left))
     )
@@
       (project "selftest_bd"
         (path "/e63e39d7-6ac0-4ffd-8aa3-1841a4541b55/3c0146c9-302b-4005-9f50-7766581fb71a"
-          (reference "K4") (unit 1)
+          (reference "K15") (unit 1)
         )
       )
@@
   (symbol (lib_id "Library:TQ2-5_Split") (at 85.09 139.7 0) (unit 1)
     (in_bom yes) (on_board yes) (dnp no)
-    (property "Reference" "K14" (at 91.44 138.4299 0)
+    (property "Reference" "K10" (at 91.44 138.4299 0)
       (effects (font (size 1.27 1.27)) (justify left))
     )
@@
       (project "selftest_bd"
         (path "/e63e39d7-6ac0-4ffd-8aa3-1841a4541b55/3c0146c9-302b-4005-9f50-7766581fb71a"
-          (reference "K14") (unit 1)
+          (reference "K10") (unit 1)
         )
       )
@@
   (symbol (lib_id "Library:TQ2-5_Split") (at 137.16 83.82 0) (unit 1)
     (in_bom yes) (on_board yes) (dnp no)
-    (property "Reference" "K10" (at 143.51 82.5499 0)
+    (property "Reference" "K13" (at 143.51 82.5499 0)
       (effects (font (size 1.27 1.27)) (justify left))
     )
@@
       (project "selftest_bd"
         (path "/e63e39d7-6ac0-4ffd-8aa3-1841a4541b55/3c0146c9-302b-4005-9f50-7766581fb71a"
-          (reference "K10") (unit 1)
+          (reference "K13") (unit 1)
         )
       )
@@
   (symbol (lib_id "Library:TQ2-5_Split") (at 116.84 83.82 0) (unit 1)
     (in_bom yes) (on_board yes) (dnp no)
-    (property "Reference" "K3" (at 123.19 82.5499 0)
+    (property "Reference" "K9" (at 123.19 82.5499 0)
       (effects (font (size 1.27 1.27)) (justify left))
     )
@@
       (project "selftest_bd"
         (path "/e63e39d7-6ac0-4ffd-8aa3-1841a4541b55/3c0146c9-302b-4005-9f50-7766581fb71a"
-          (reference "K3") (unit 1)
+          (reference "K9") (unit 1)
         )
       )
@@
   (symbol (lib_id "Library:TQ2-5_Split") (at 157.48 83.82 0) (unit 1)
     (in_bom yes) (on_board yes) (dnp no)
-    (property "Reference" "K11" (at 163.83 82.5499 0)
+    (property "Reference" "K6" (at 163.83 82.5499 0)
       (effects (font (size 1.27 1.27)) (justify left))
     )
@@
       (project "selftest_bd"
         (path "/e63e39d7-6ac0-4ffd-8aa3-1841a4541b55/3c0146c9-302b-4005-9f50-7766581fb71a"
-          (reference "K11") (unit 1)
-        )
-      )
+          (reference "K6") (unit 1)
+        )
+      )

Commit message: update README and small correction
Connections:
- net PM1_IO8 renamed PM1_IO0
- net PM1_IO9 renamed PM1_IO1
Other:
- title: FIRST TEST STATION SELFTEST BOARD 640-1010-020 -> FIRST TEST STATION SELFTEST BOARD 640-1010-021
Changed lines of the file:
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@@
   (paper "A")
   (title_block
-    (title "FIRST TEST STATION SELFTEST BOARD 640-1010-020")
+    (title "FIRST TEST STATION SELFTEST BOARD 640-1010-021")
     (date "2023-10-01")
-    (rev "2.0")
+    (rev "2.1")
   )
   (junction (at 110.49 147.32) (diameter 0) (color 0 0 0 0)
@@
     )
   )
-  (global_label "PM1_IO8" (shape bidirectional) (at 30.48 95.25 180) (fields_autoplaced)
-    (effects (font (size 1.27 1.27)) (justify right))
-    (property "Intersheetrefs" "${INTERSHEET_REFS}" (at 20.0236 95.1706 0)
+  (global_label "PM1_IO0" (shape bidirectional) (at 30.48 95.25 180) (fields_autoplaced)
+    (effects (font (size 1.27 1.27)) (justify right))
+    (property "Intersheetrefs" "${INTERSHEET_REFS}" (at 18.4196 95.25 0)
       (effects (font (size 1.27 1.27)) (justify right) hide)
     )
@@
     )
   )
-  (global_label "PM1_IO9" (shape bidirectional) (at 30.48 102.87 180) (fields_autoplaced)
-    (effects (font (size 1.27 1.27)) (justify right))
-    (property "Intersheetrefs" "${INTERSHEET_REFS}" (at 20.0236 102.7906 0)
-      (effects (font (size 1.27 1.27)) (justify right) hide)
-    )
+  (global_label "PM1_IO1" (shape bidirectional) (at 30.48 102.87 180) (fields_autoplaced)
+    (effects (font (size 1.27 1.27)) (justify right))
+    (property "Intersheetrefs" "${INTERSHEET_REFS}" (at 18.4196 102.87 0)
+      (effects (font (size 1.27 1.27)) (justify right) hide)
+    )
