File: selftest_bd/selftest_bd.kicad_sch (KiCad schematic)
At the start: 0 parts

Commit message: Commit V2.0
Redo PCB due to incorrect position of J1 and J2
Other:
- title: FIRST TEST STATION SELFTEST BOARD 640-1010-010 -> FIRST TEST STATION SELFTEST BOARD 640-1010-020
Changed lines of the file:
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@@
   (paper "A")
   (title_block
-    (title "FIRST TEST STATION SELFTEST BOARD 640-1010-010")
-    (date "2023-05-16")
-    (rev "1.0")
+    (title "FIRST TEST STATION SELFTEST BOARD 640-1010-020")
+    (date "2023-10-01")
+    (rev "2.0")
   )
   (image (at 201.93 179.07) (scale 2.13772)

Commit message: update README and small correction
Other:
- title: FIRST TEST STATION SELFTEST BOARD 640-1010-020 -> FIRST TEST STATION SELFTEST BOARD 640-1010-021
Changed lines of the file:
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@@
   (paper "A")
   (title_block
-    (title "FIRST TEST STATION SELFTEST BOARD 640-1010-020")
+    (title "FIRST TEST STATION SELFTEST BOARD 640-1010-021")
     (date "2023-10-01")
-    (rev "2.0")
+    (rev "2.1")
   )
   (image (at 201.93 179.07) (scale 2.13772)
