File: selftest_bd/test_connector.kicad_sch (KiCad schematic)
At the start: 45 parts, among them J3 RJ45, J4 USB-VERTICAL, J5 8 x 2.54mm, J6 8 x 2.54mm, U4 11AA10, U5 11AA10

Commit message: Commit V2.0
Redo PCB due to incorrect position of J1 and J2
Parts:
- C3: footprint Capacitor_THT:CP_Radial_D4.0mm_P1.50mm -> Capacitor_THT:CP_Radial_Tantal_D4.5mm_P2.50mm
- R13, R14: value 4.7K -> 1K
- R15: value 220 -> 470
- R16: value 120 -> 330
- U4, U5: value 11AA10 -> DS2431; footprint Package_TO_SOT_THT:TO-92_Inline -> Package_TO_SOT_THT:TO-92_HandSolder
Other:
- note added: "RED"
- title: FIRST TEST STATION SELFTEST BOARD 640-1010-010 -> FIRST TEST STATION SELFTEST BOARD 640-1010-020
Changed lines of the file:
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@@
   (paper "A")
   (title_block
-    (title "FIRST TEST STATION SELFTEST BOARD 640-1010-010")
-    (date "2023-05-16")
-    (rev "1.0")
+    (title "FIRST TEST STATION SELFTEST BOARD 640-1010-020")
+    (date "2023-10-01")
+    (rev "2.0")
   )
   (junction (at 109.22 182.88) (diameter 0) (color 0 0 0 0)
@@
     (effects (font (size 1.27 1.27)) (justify left bottom))
   )
-  (text "GREEN" (at 165.1 115.57 0)
+  (text "RED" (at 165.1 115.57 0)
     (effects (font (size 1.27 1.27)) (justify left bottom))
   )
@@
       (effects (font (size 1.27 1.27)))
     )
-    (property "Value" "11AA10" (at 137.16 148.59 0)
+    (property "Value" "DS2431" (at 137.16 148.59 0)
       (effects (font (size 1.27 1.27)))
     )
-    (property "Footprint" "Package_TO_SOT_THT:TO-92_Inline" (at 137.16 156.21 0)
+    (property "Footprint" "Package_TO_SOT_THT:TO-92_HandSolder" (at 137.16 156.21 0)
       (effects (font (size 1.27 1.27)) (justify bottom) hide)
     )
@@
       (effects (font (size 1.27 1.27)))
     )
-    (property "Value" "4.7K" (at 113.03 172.72 0)
+    (property "Value" "1K" (at 113.03 172.72 0)
       (effects (font (size 1.27 1.27)))
     )
@@
       (effects (font (size 1.27 1.27)))
     )
-    (property "Value" "11AA10" (at 137.16 177.8 0)
+    (property "Value" "DS2431" (at 137.16 177.8 0)
       (effects (font (size 1.27 1.27)))
     )
-    (property "Footprint" "Package_TO_SOT_THT:TO-92_Inline" (at 137.16 185.42 0)
+    (property "Footprint" "Package_TO_SOT_THT:TO-92_HandSolder" (at 137.16 185.42 0)
       (effects (font (size 1.27 1.27)) (justify bottom) hide)
     )
@@
       (effects (font (size 1.27 1.27)) (justify left))
     )
-    (property "Footprint" "Capacitor_THT:CP_Radial_D4.0mm_P1.50mm" (at 152.0952 59.69 0)
+    (property "Footprint" "Capacitor_THT:CP_Radial_Tantal_D4.5mm_P2.50mm" (at 152.0952 59.69 0)
       (effects (font (size 1.27 1.27)) hide)
     )
@@
       (effects (font (size 1.27 1.27)))
     )
-    (property "Value" "120" (at 222.25 99.06 90)
+    (property "Value" "330" (at 222.25 99.06 90)
       (effects (font (size 1.27 1.27)))
     )
@@
       (effects (font (size 1.27 1.27)))
     )
-    (property "Value" "220" (at 165.1 99.06 90)
+    (property "Value" "470" (at 165.1 99.06 90)
       (effects (font (size 1.27 1.27)))
     )
@@
       (effects (font (size 1.27 1.27)))
     )
-    (property "Value" "4.7K" (at 113.03 143.51 0)
+    (property "Value" "1K" (at 113.03 143.51 0)
       (effects (font (size 1.27 1.27)))
     )

Commit message: update README and small correction
Parts:
- R13, R14: value 1K -> N.A
Connections:
- net ETH_RX+: now also J3.3; no longer J3.6
- net ETH_RX-: now also J3.6; no longer J3.3
- net ETH_TX+: now also J3.1; no longer J3.8
- net ETH_TX-: now also J3.2; no longer J3.7
- net USB_D+: now also J4.3 (D+); no longer J4.2 (D-)
- net USB_D-: now also J4.2 (D-); no longer J4.3 (D+)
- net at TP23.1: now also J3.8; no longer J3.2
- net at TP22.1: now also J3.7; no longer J3.1
Other:
- note added: "N.A NOT ASSEMBLED"
- title: FIRST TEST STATION SELFTEST BOARD 640-1010-020 -> FIRST TEST STATION SELFTEST BOARD 640-1010-021
- moved on the sheet: TP22, TP23, TP24, TP25
